File: power.kicad_sch (KiCad schematic)
At the start: 1 part, among them J201 USB_C_Receptacle_USB2.0

Commit message: Finished cconnections for imu
Parts:
- removed J201: USB_C_Receptacle_USB2.0, symbol Connector:USB_C_Receptacle_USB2.0
Changed lines of the file:
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@@
 (kicad_sch (version 20230121) (generator eeschema)
   (paper "A4")
-  (symbol (lib_id "Connector:USB_C_Receptacle_USB2.0") (at 43.18 66.04 0) (unit 1)
-    (in_bom yes) (on_board yes) (dnp no) (fields_autoplaced)
-    (property "Reference" "J201" (at 43.18 43.18 0)
-      (effects (font (size 1.27 1.27)))
-    )
-    (property "Value" "USB_C_Receptacle_USB2.0" (at 43.18 45.72 0)
-      (effects (font (size 1.27 1.27)))
-    )
-    (property "Footprint" "" (at 46.99 66.04 0)
-      (effects (font (size 1.27 1.27)) hide)
-    )
-    (property "Datasheet" "https://www.usb.org/sites/default/files/documents/usb_type-c.zip" (at 46.99 66.04 0)
-      (effects (font (size 1.27 1.27)) hide)
-    )
-    (pin "A1")
-    (pin "A12")
-    (pin "A4")
-    (pin "A5")
-    (pin "A6")
-    (pin "A7")
-    (pin "A8")
-    (pin "A9")
-    (pin "B1")
-    (pin "B12")
-    (pin "B4")
-    (pin "B5")
-    (pin "B6")
-    (pin "B7")
-    (pin "B8")
-    (pin "B9")
-    (pin "S1")
-    (instances
-      (project "MicroQuad"
-        (path "/8971f876-5b3c-4165-aa17-84d4a3cd004e/6efdce62-27dc-4b15-aeb6-b54c510c1d4f"
-          (reference "J201") (unit 1)
-        )
-      )
-    )
-  )
 )

Commit message: Added some components
Parts:
- added J201: USB_C_Receptacle_USB2.0, symbol Connector:USB_C_Receptacle_USB2.0
Connections:
- new net: J201.A1 (GND), J201.A12 (GND), J201.B1 (GND), J201.B12 (GND)
- new net: J201.A4 (VBUS), J201.A9 (VBUS), J201.B4 (VBUS), J201.B9 (VBUS)
Changed lines of the file:
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@@
 (kicad_sch (version 20230121) (generator eeschema)
   (paper "A4")
+  (symbol (lib_id "Connector:USB_C_Receptacle_USB2.0") (at 43.18 66.04 0) (unit 1)
+    (in_bom yes) (on_board yes) (dnp no) (fields_autoplaced)
+    (property "Reference" "J201" (at 43.18 43.18 0)
+      (effects (font (size 1.27 1.27)))
+    )
+    (property "Value" "USB_C_Receptacle_USB2.0" (at 43.18 45.72 0)
+      (effects (font (size 1.27 1.27)))
+    )
+    (property "Footprint" "" (at 46.99 66.04 0)
+      (effects (font (size 1.27 1.27)) hide)
+    )
+    (property "Datasheet" "https://www.usb.org/sites/default/files/documents/usb_type-c.zip" (at 46.99 66.04 0)
+      (effects (font (size 1.27 1.27)) hide)
+    )
+    (pin "A1")
+    (pin "A12")
+    (pin "A4")
+    (pin "A5")
+    (pin "A6")
+    (pin "A7")
+    (pin "A8")
+    (pin "A9")
+    (pin "B1")
+    (pin "B12")
+    (pin "B4")
+    (pin "B5")
+    (pin "B6")
+    (pin "B7")
+    (pin "B8")
+    (pin "B9")
+    (pin "S1")
+    (instances
+      (project "MicroQuad"
+        (path "/8971f876-5b3c-4165-aa17-84d4a3cd004e/6efdce62-27dc-4b15-aeb6-b54c510c1d4f"
+          (reference "J201") (unit 1)
+        )
+      )
+    )
+  )
 )
